Commit message: feat(retargeting): add rubber-hand A1 wrist pipeline

File: src/holosoma/holosoma/data/robots/g1/main_mesh_collision_rubberhand.urdf (robot description, URDF)
Before this commit: robot g1, 42 links, 41 joints
Links:
- removed link left_sphere_hand_link
- removed link right_sphere_hand_link
- added link left_rubber_hand_link, mass 0.170; collision mesh filename=meshes/left_rubber_hand.STL; visual mesh filename=meshes/left_rubber_hand.STL
- added link right_rubber_hand_link, mass 0.170; collision mesh filename=meshes/right_rubber_hand.STL; visual mesh filename=meshes/right_rubber_hand.STL
Joints:
- joint left_hand_palm_joint: child left_sphere_hand_link -> left_rubber_hand_link; origin xyz=0.029 -0.003 0 rpy=0 1.57 0 -> xyz=0.0415 0.003 0 rpy=0 0 0
- joint right_hand_palm_joint: child right_sphere_hand_link -> right_rubber_hand_link; origin xyz=0.029 -0.003 0 rpy=0 1.57 0 -> xyz=0.0415 -0.003 0 rpy=0 0 0
